Commit message: se añadieron notas de clase hasta clase 21

File: moveit2_ws/install/my_robot_description/share/my_robot_description/urdf/arm.xacro (robot description, xacro)
@@ -9,4 +9,10 @@
             </geometry>
         </visual>
+        <collision>
+            <origin xyz="0 0 0.05" rpy="0 0 0" />
+            <geometry>
+                <box size="0.4 0.4 0.1"  />
+            </geometry>
+        </collision>
     </link>
     <link name="shoulder_link">
@@ -18,4 +24,10 @@
             <material name="blue" />
         </visual>
+        <collision>
+            <origin xyz="0 0 0.25" rpy="0 0 0" />
+            <geometry>
+                <cylinder length="0.5" radius="0.1" />
+            </geometry>
+        </collision>
     </link>
     <link name="arm_link">
@@ -27,4 +39,10 @@
             <material name="grey" />
         </visual>
+        <collision>
+            <origin xyz="0 0 0.3" rpy="0 0 0" />
+            <geometry>
+                <cylinder radius="0.05" length="0.6" />
+            </geometry>
+        </collision>
     </link>
     <link name="elbow_link">
@@ -36,4 +54,10 @@
             <material name="blue" />
         </visual>
+        <collision>
+            <origin xyz="0 0 0.05" rpy="0 0 0" />
+            <geometry>
+                <cylinder radius="0.05" length="0.1" />
+            </geometry>
+        </collision>
     </link>
     <link name="forearm_link">
@@ -45,4 +69,10 @@
             <material name="grey" />
         </visual>
+        <collision>
+            <origin xyz="0 0 0.25" rpy="0 0 0" />
+            <geometry>
+                <cylinder radius="0.05" length="0.5" />
+            </geometry>
+        </collision>
     </link>
     <link name="wrist_link">
@@ -54,4 +84,10 @@
             <material name="blue" />
         </visual>
+        <collision>
+            <origin xyz="0 0 0.025" rpy="0 0 0" />
+            <geometry>
+                <box size="0.1 0.1 0.05" />
+            </geometry>
+        </collision>
     </link>
     <link name="hand_link">
@@ -63,4 +99,10 @@
             <material name="grey" />
         </visual>
+        <collision>
+            <origin xyz="0 0 0.01" rpy="0 0 0" />
+            <geometry>
+                <box size="0.1 0.1 0.02" />
+            </geometry>
+        </collision>
     </link>
     <link name="hand_tool_link">

Commit message: se añadieron notas de clase hasta clase 27

File: moveit2_ws/install/my_robot_description/share/my_robot_description/urdf/arm.xacro (robot description, xacro)
@@ -106,5 +106,5 @@
         </collision>
     </link>
-    <link name="hand_tool_link">
+    <link name="tool_link">
     </link>
     <joint name="joint1" type="revolute">
@@ -152,5 +152,5 @@
     <joint name="hand_tool_joint" type="fixed">
         <parent link="hand_link" />
-        <child link="hand_tool_link" />
+        <child link="tool_link" />
         <origin xyz="0 0 0.02" rpy="0 0 0" />
     </joint>

File: moveit2_ws/install/my_robot_description/share/my_robot_description/urdf/my_robot.urdf.xacro (robot description, xacro)
@@ -3,3 +3,9 @@
     <xacro:include filename="common_properties.xacro" />
     <xacro:include filename="arm.xacro"/>
+    <xacro:include filename="gripper.xacro"/>
+    <joint name="gripper_base_joint" type="fixed">
+        <parent link="tool_link" />
+        <child link="gripper_base_link" />
+        <origin xyz="0 0 0" rpy="0 0 0" />
+    </joint>
 </robot>
